File: schematics/batteryTester/batteryTester.sch (KiCad schematic (older format))
At the start: 8 parts

Commit message: update schematic (incomplete)
Parts:
- added D?: DIODE, symbol pspice:DIODE
- added J?: Battery to test, symbol Connector:Barrel_Jack
- added R?: 86k, symbol Device:R
- added R?: 10k, symbol Device:R
- added R?: 15k, symbol Device:R
- added R? (x2): 1k, symbol Device:R
- added R?: 0.1, symbol Device:R
- added R?: 1.5, symbol Device:R
Connections:
- net GND: now also J?.2, R?.2, R?.2, R?.2; no longer U?.6 (GND)
- net at U?.2 (SCL): no longer U?.4 (SCL)
- net at U?.3 (SDA): no longer U?.3 (SDA)
- net at U?.6 (VOUTA): now also U?.5 (+)
- net at U?.7 (IN-): now also D?.1 (K)
- net at U?.8 (IN+): now also J?.1
- net at U?.1: now also Q?.1 (G), R?.1, R?.1
- net at U?.2 (-): now also R?.1, R?.2
- net at U?.3 (+): now also R?.1, R?.1
- net at U?.6 (-): now also U?.7, R?.2
- net at Q?.2 (D): now also R?.2
- net at Q?.3 (S): now also R?.1, R?.2
- new net: D?.2 (A), R?.1
Other:
- moved on the sheet: Q?, SW?, U?, U?A, U?B

Commit message: update kicad schematic
Connections:
- wire segments 72 -> 88
Changed lines of the file:
@@
 Wire Wire Line
 	9100 1050 9450 1050
+Wire Wire Line
+	4850 950  1150 950
+Wire Wire Line
+	1150 950  1150 4050
+Wire Wire Line
+	1150 4050 1350 4050
+Wire Wire Line
+	4850 2200 4750 2200
+Wire Wire Line
+	4750 2200 4750 1300
+Wire Wire Line
+	4750 1050 1300 1050
+Wire Wire Line
+	1300 1050 1300 4150
+Wire Wire Line
+	1300 4150 1350 4150
+Wire Wire Line
+	8200 1000 8150 1000
+Wire Wire Line
+	4850 950  4850 1000
+Connection ~ 4850 1000
+Wire Wire Line
+	4850 1000 4850 2100
+Connection ~ 8150 1000
+Wire Wire Line
+	8150 1000 4850 1000
+Wire Wire Line
+	5150 900  5150 1300
+Wire Wire Line
+	5150 1300 4750 1300
+Wire Wire Line
+	5150 900  8150 900
+Connection ~ 4750 1300
+Wire Wire Line
+	4750 1300 4750 1050
 $EndSCHEMATC

Commit message: update schematic with touchscreen, even if we dont really use it
Parts:
- added U?: XPT2046TS, Package_SO:TSSOP-16_4.4x5mm_P0.65mm, symbol Driver_Display:XPT2046TS
Connections:
- wire segments 88 -> 106
Other:
- moved on the sheet: D?, J?, Q?, R?, SW?, U?, U?A, U?B
