File: schematics/batteryTesterLc/tester.sch (KiCad schematic (older format))
At the start: 44 parts, among them J1 UART, J2 Probes, J3 USB_B_Micro, J4 ST7735, SW1 Rotary_Encoder_Switch, U1 STM32F103C8Tx, U2 LMV324, U3 LM324, U4 AMS1117-3.3, Y1 8Mhz

Commit message: use adc as submodule
Parts:
- removed C11: 100nF, symbol pspice:C
- removed C9: 100nF, symbol pspice:CAP
- removed D1: LED, symbol Device:LED
- removed J1: UART, symbol Connector:Conn_01x02_Male
- removed J2: Probes, symbol Connector:Conn_01x03_Female
- removed J4: ST7735, symbol Connector:Conn_01x08_Female
- removed R10, R17, R8: 0, symbol Device:R
- removed R11, R15, R5: 470, symbol Device:R
- removed R12, R14, R7: 470k, symbol Device:R
- removed R13, R16, R6: 15k, symbol Device:R
- removed R18: 150k, symbol Device:R_Small_US
- removed R19: 4.7k, symbol Device:R_Small
- removed R20, R21: 20, symbol Device:R_Small
- removed R4: 510, symbol Device:R_Small_US
- removed U2, U?: LMV324, symbol Amplifier_Operational:LMV324
- removed U3: LM324, symbol Amplifier_Operational:LM324
- added C?: 33uF, symbol pspice:C
- added C? (x2): 100nF, symbol pspice:C
- added D?: BLUE LED (2.5v), symbol Device:LED_ALT
- added Q?: AO3401A, Package_TO_SOT_SMD:SOT-23, symbol Transistor_FET:AO3401A
- added R? (x2): 20k, symbol Device:R_Small
- added U?: CR2013-MI2120, Display:CR2013-MI2120, symbol Driver_Display:CR2013-MI2120
- added U?: XPT2046QF, Package_DFN_QFN:QFN-16-1EP_4x4mm_P0.65mm_EP2.1x2.1mm, symbol Driver_Display:XPT2046QF
Connections:
- net labels added: BAT+, BAT-, LCDCS, LCDDC, LCDRST, SPI1CLK, SPI1MISO, SPI1MOSI, SWDCLK, SWDIO, TOUCH_CS, TOUCH_IRQ, UART1TX, VBATSENSE
- net labels removed: A0, CS, LED, RST, SCK, SDA, VCC
- wire segments 204 -> 146
Other:
- note removed: "PA0\n"
- note removed: "PA1"
- note removed: "PA2"
- note removed: "RX"
- note removed: "TX"
- moved on the sheet: C1, C10, C2, C3, C4, C5, C6, C7, C8, R1, R2, R3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

Commit message: update adc
Parts:
- added C1, C2: 330n, symbol Device:C_Small
- added R1, R2: 20k, symbol Device:R_Small_US
- gave numbers to parts that had none: 9
- renumbered C1 to C10, C2 to C12, C3 to C14, C5 to C3, C6 to C4, C7 to C5, C8 to C6, C4 to C7, C10 to C9, J3 to J1, R9 to R3, R1 to R6, R2 to R7, R3 to R8, U1 to U2
Connections:
- net labels added: GATECONTROL
- wire segments 146 -> 153

Commit message: sync with demo code
Parts:
- removed C10, C12, C14: CAP, symbol pspice:CAP
- removed R6: R_Small, symbol Device:R_Small
- removed SW1: Rotary_Encoder_Switch, symbol Device:Rotary_Encoder_Switch
- removed U1: CR2013-MI2120, Display:CR2013-MI2120, symbol Driver_Display:CR2013-MI2120
- removed U3: XPT2046QF, Package_DFN_QFN:QFN-16-1EP_4x4mm_P0.65mm_EP2.1x2.1mm, symbol Driver_Display:XPT2046QF
- added C8: 100n, symbol Device:C
- added J2: Conn_01x02_Male, symbol Connector:Conn_01x02_Male
- added J?: Conn_01x05, symbol Connector_Generic:Conn_01x05
- added J?: Conn_01x04, symbol Connector_Generic:Conn_01x04
- added M1: MNMOS, symbol pspice:MNMOS
- added Q2: AO3401A, Package_TO_SOT_SMD:SOT-23, symbol Transistor_FET:AO3401A
- added Q?: Q_NPN_BCE, symbol Device:Q_NPN_BCE
- added R10: 820, symbol Device:R_Small
- added R11: 2.4, symbol Device:R_Small
- added R12: 0.1, symbol Device:R_Small
- added R13, R9: 10k, symbol Device:R_Small
- added R4: 470k, symbol Device:R_Small
- added R?: 150k....180k, symbol Device:R_Small
- added R?: 1k, symbol Device:R_Small
- added U4: LMV324, symbol Amplifier_Operational:LMV324
- J1: symbol Connector:USB_B_Micro -> tester-rescue:USB_B_Micro-Connector
- R7: value R_Small -> 1k
- R8: value R_Small -> 22k
- renumbered C8 to C10, C9 to C11, C11 to C13, C13 to C15, R4 to R5, R5 to R6, U4 to U5
Connections:
- net labels added: BAT_ENABLE, ISENSE, PWM
- wire segments 153 -> 164
Other:
- note added: "D"
- note added: "S"
- moved on the sheet: C1, C10, C11, C13, C15, C2, C3, C4, C5, C6, C7, D1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

Commit message: sync with Arduino_stm32
Parts:
- removed Q2: AO3401A, Package_TO_SOT_SMD:SOT-23, symbol Transistor_FET:AO3401A
- removed Q?: Q_NPN_BCE, symbol Device:Q_NPN_BCE
- removed R4: 470k, symbol Device:R_Small
- removed R?: 1k, symbol Device:R_Small
- added D?: DIODE, symbol pspice:DIODE
Connections:
- wire segments 164 -> 156
Other:
- moved on the sheet: D1, J2, Q1, R5, R6

Commit message: update schematic
Parts:
- added RVX, RVY: R_POT, symbol Device:R_POT
- added SW?: Joystick, symbol Switch:SW_Push
- J1: symbol tester-rescue:USB_B_Micro-Connector -> tester-rescue:USB_B_Micro-Connector-tester-rescue
Connections:
- wire segments 156 -> 175
Changed lines of the file:
@@
 	3550 1950 3550 1900
 $Comp
-L tester-rescue:USB_B_Micro-Connector J1
+L tester-rescue:USB_B_Micro-Connector-tester-rescue J1
 U 1 1 5E792D53
 P 10000 1400
@@
 Wire Wire Line
 	7050 900  7050 2000
+$Comp
+L Device:R_POT RVY
+U 1 1 61D8C54E
+P 4250 2750
+F 0 "RVY" H 4180 2796 50  0000 R CNN
+F 1 "R_POT" H 4180 2705 50  0000 R CNN
+F 2 "" H 4250 2750 50  0001 C CNN
+F 3 "~" H 4250 2750 50  0001 C CNN
+	1    4250 2750
+	-1   0    0    -1
+$EndComp
+$Comp
+L Device:R_POT RVX
+U 1 1 61D948C4
+P 4900 2750
+F 0 "RVX" H 4830 2796 50  0000 R CNN
+F 1 "R_POT" H 4830 2705 50  0000 R CNN
+F 2 "" H 4900 2750 50  0001 C CNN
+F 3 "~" H 4900 2750 50  0001 C CNN
+	1    4900 2750
+	-1   0    0    -1
+$EndComp
+$Comp
+L power:+3.3V #PWR?
+U 1 1 61D97E3F
+P 4050 2550
+F 0 "#PWR?" H 4050 2400 50  0001 C CNN
+F 1 "+3.3V" H 4065 2723 50  0000 C CNN
+F 2 "" H 4050 2550 50  0001 C CNN
+F 3 "" H 4050 2550 50  0001 C CNN
+	1    4050 2550
+	1    0    0    -1
+$EndComp
+$Comp
+L power:GND #PWR?
+U 1 1 61D98F30
+P 4500 3000
+F 0 "#PWR?" H 4500 2750 50  0001 C CNN
+F 1 "GND" H 4505 2827 50  0000 C CNN
+F 2 "" H 4500 3000 50  0001 C CNN
+F 3 "" H 4500 3000 50  0001 C CNN
+	1    4500 3000
+	1    0    0    -1
+$EndComp
+Wire Wire Line
+	4050 2550 4050 2600
+Wire Wire Line
+	4050 2600 4250 2600
+Connection ~ 4250 2600
+Wire Wire Line
+	4250 2600 4900 2600
+Wire Wire Line
+	4250 2900 4500 2900
+Wire Wire Line
+	4500 2900 4500 3000
+Connection ~ 4500 2900
+Wire Wire Line
+	4500 2900 4900 2900
+Wire Wire Line
+	4100 2750 3850 2750
+Wire Wire Line
+	3850 2750 3850 3500
+Wire Wire Line
+	3850 3500 3550 3500
+Wire Wire Line
+	4750 2750 4750 3600
+Wire Wire Line
+	4750 3600 3550 3600
+$Comp
+L Switch:SW_Push SW?
+U 1 1 61DC3EAE
+P 5400 2700
+F 0 "SW?" V 5354 2848 50  0000 L CNN
+F 1 "Joystick" V 5445 2848 50  0000 L CNN
+F 2 "" H 5400 2900 50  0001 C CNN
+F 3 "~" H 5400 2900 50  0001 C CNN
+	1    5400 2700
+	0    1    1    0
+$EndComp
+Wire Wire Line
+	4900 2900 5400 2900
+Connection ~ 4900 2900
+Wire Wire Line
+	2250 3500 3100 3500
+Wire Wire Line
+	3100 3500 3100 2800
+Wire Wire Line
+	3100 2800 3700 2800
+Wire Wire Line
+	3700 2800 3700 2200
+Wire Wire Line
+	3700 2200 4750 2200
+Wire Wire Line
+	4750 2200 4750 2500
+Wire Wire Line
+	4750 2500 5400 2500
 $EndSCHEMATC

Commit message: sync
Parts:
- removed RVX, RVY: R_POT, symbol Device:R_POT
- added SW?: Down, symbol Switch:SW_Push
- added SW?: Left, symbol Switch:SW_Push
- added SW?: Right, symbol Switch:SW_Push
- added SW?: Up, symbol Switch:SW_Push
- J1: symbol tester-rescue:USB_B_Micro-Connector-tester-rescue -> tester-rescue:USB_B_Micro-Connector-tester-rescue-tester-rescue
- SW?: value Joystick -> Button
Connections:
- wire segments 175 -> 183
Other:
- moved on the sheet: SW?
Changed lines of the file:
@@
 	3550 1950 3550 1900
 $Comp
-L tester-rescue:USB_B_Micro-Connector-tester-rescue J1
+L tester-rescue:USB_B_Micro-Connector-tester-rescue-tester-rescue J1
 U 1 1 5E792D53
 P 10000 1400
@@
 	1    1600 2600
 	0    1    1    0
-$EndComp
-Connection ~ 2950 2100
-Connection ~ 2750 2100
-Wire Wire Line
-	2550 2100 2750 2100
-Connection ~ 2850 2100
-Wire Wire Line
-	2750 2100 2850 2100
-Wire Wire Line
-	2850 2100 2950 2100
-Connection ~ 2850 5100
-Wire Wire Line
-	2750 5100 2850 5100
-Wire Wire Line
-	2850 5100 2950 5100
-Connection ~ 2950 5100
-Connection ~ 3050 5100
-Wire Wire Line
-	2950 5100 3050 5100
-Wire Wire Line
-	3300 5100 3050 5100
-$Comp
-L MCU_ST_STM32F1:STM32F103C8Tx U2
-U 1 1 5E490CEE
-P 2950 3600
-F 0 "U2" H 2900 2014 50  0000 C CNN
-F 1 "STM32F103C8Tx" H 2900 1923 50  0000 C CNN
-F 2 "Package_QFP:LQFP-48_7x7mm_P0.5mm" H 2350 2200 50  0001 R CNN
-F 3 "" H 2950 3600 50  0001 C CNN
-	1    2950 3600
-	1    0    0    -1
 $EndComp
 Wire Wire Line
@@
 	7050 900  7050 2000
 $Comp
-L Device:R_POT RVY
-U 1 1 61D8C54E
-P 4250 2750
-F 0 "RVY" H 4180 2796 50  0000 R CNN
-F 1 "R_POT" H 4180 2705 50  0000 R CNN
-F 2 "" H 4250 2750 50  0001 C CNN
-F 3 "~" H 4250 2750 50  0001 C CNN
-	1    4250 2750
-	-1   0    0    -1
-$EndComp
-$Comp
-L Device:R_POT RVX
-U 1 1 61D948C4
-P 4900 2750
-F 0 "RVX" H 4830 2796 50  0000 R CNN
-F 1 "R_POT" H 4830 2705 50  0000 R CNN
-F 2 "" H 4900 2750 50  0001 C CNN
-F 3 "~" H 4900 2750 50  0001 C CNN
-	1    4900 2750
-	-1   0    0    -1
-$EndComp
-$Comp
-L power:+3.3V #PWR?
-U 1 1 61D97E3F
-P 4050 2550
-F 0 "#PWR?" H 4050 2400 50  0001 C CNN
-F 1 "+3.3V" H 4065 2723 50  0000 C CNN
-F 2 "" H 4050 2550 50  0001 C CNN
-F 3 "" H 4050 2550 50  0001 C CNN
-	1    4050 2550
-	1    0    0    -1
-$EndComp
-$Comp
 L power:GND #PWR?
 U 1 1 61D98F30
-P 4500 3000
-F 0 "#PWR?" H 4500 2750 50  0001 C CNN
-F 1 "GND" H 4505 2827 50  0000 C CNN
-F 2 "" H 4500 3000 50  0001 C CNN
-F 3 "" H 4500 3000 50  0001 C CNN
-	1    4500 3000
+P 4750 3350
+F 0 "#PWR?" H 4750 3100 50  0001 C CNN
+F 1 "GND" H 4755 3177 50  0000 C CNN
+F 2 "" H 4750 3350 50  0001 C CNN
+F 3 "" H 4750 3350 50  0001 C CNN
+	1    4750 3350
 	1    0    0    -1
 $EndComp
 Wire Wire Line
 	4050 2550 4050 2600
-Wire Wire Line
-	4050 2600 4250 2600
-Connection ~ 4250 2600
-Wire Wire Line
-	4250 2600 4900 2600
-Wire Wire Line
-	4250 2900 4500 2900
-Wire Wire Line
-	4500 2900 4500 3000
-Connection ~ 4500 2900
-Wire Wire Line
-	4500 2900 4900 2900
-Wire Wire Line
-	4100 2750 3850 2750
-Wire Wire Line
-	3850 2750 3850 3500
-Wire Wire Line
-	3850 3500 3550 3500
-Wire Wire Line
-	4750 2750 4750 3600
-Wire Wire Line
-	4750 3600 3550 3600
 $Comp
 L Switch:SW_Push SW?
 U 1 1 61DC3EAE
-P 5400 2700
-F 0 "SW?" V 5354 2848 50  0000 L CNN
-F 1 "Joystick" V 5445 2848 50  0000 L CNN
-F 2 "" H 5400 2900 50  0001 C CNN
-F 3 "~" H 5400 2900 50  0001 C CNN
-	1    5400 2700
+P 5450 3000
+F 0 "SW?" V 5750 2900 50  0000 L CNN
+F 1 "Button" V 5750 3050 50  0000 L CNN
+F 2 "" H 5450 3200 50  0001 C CNN
+F 3 "~" H 5450 3200 50  0001 C CNN
+	1    5450 3000
 	0    1    1    0
 $EndComp
 Wire Wire Line
-	4900 2900 5400 2900
-Connection ~ 4900 2900
-Wire Wire Line
-	2250 3500 3100 3500
-Wire Wire Line
-	3100 3500 3100 2800
-Wire Wire Line
-	3100 2800 3700 2800
-Wire Wire Line
-	3700 2800 3700 2200
-Wire Wire Line
-	3700 2200 4750 2200
-Wire Wire Line
-	4750 2200 4750 2500
-Wire Wire Line
-	4750 2500 5400 2500
+	2250 3500 2650 3500
+$Comp
+L Switch:SW_Push SW?
+U 1 1 61E3421F
+P 4100 3000
+F 0 "SW?" V 4054 3148 50  0000 L CNN
+F 1 "Down" V 4145 3148 50  0000 L CNN
+F 2 "" H 4100 3200 50  0001 C CNN
+F 3 "~" H 4100 3200 50  0001 C CNN
+	1    4100 3000
+	0    1    1    0
+$EndComp
+$Comp
+L Switch:SW_Push SW?
+U 1 1 61E3B4A0
+P 4550 3000
+F 0 "SW?" V 4800 2800 50  0000 L CNN
+F 1 "Left" V 4800 3000 50  0000 L CNN
+F 2 "" H 4550 3200 50  0001 C CNN
+F 3 "~" H 4550 3200 50  0001 C CNN
+	1    4550 3000
+	0    1    1    0
+$EndComp
+$Comp
+L Switch:SW_Push SW?
+U 1 1 61E3C424
+P 4950 3000
+F 0 "SW?" V 4904 3148 50  0000 L CNN
+F 1 "Right" V 4995 3148 50  0000 L CNN
+F 2 "" H 4950 3200 50  0001 C CNN
+F 3 "~" H 4950 3200 50  0001 C CNN
+	1    4950 3000
+	0    1    1    0
+$EndComp
+$Comp
+L Switch:SW_Push SW?
+U 1 1 61E3D547
+P 3850 3000
+F 0 "SW?" V 4150 2850 50  0000 L CNN
+F 1 "Up" V 4150 3000 50  0000 L CNN
+F 2 "" H 3850 3200 50  0001 C CNN
+F 3 "~" H 3850 3200 50  0001 C CNN
+	1    3850 3000
+	0    1    1    0
+$EndComp
+Wire Wire Line
+	3850 3200 4100 3200
+Wire Wire Line
+	4950 3200 4950 3350
+Wire Wire Line
+	4950 3350 4750 3350
+Connection ~ 4950 3200
+Connection ~ 4100 3200
+Wire Wire Line
+	4100 3200 4550 3200
+Connection ~ 4550 3200
+Wire Wire Line
+	4550 3200 4950 3200
+Wire Wire Line
+	3300 5100 3050 5100
+Connection ~ 3050 5100
+Wire Wire Line
+	2950 5100 3050 5100
+Connection ~ 2950 5100
+Wire Wire Line
+	2850 5100 2950 5100
+Wire Wire Line
+	2750 5100 2850 5100
+Connection ~ 2850 5100
+Connection ~ 2950 2100
+Wire Wire Line
+	2850 2100 2950 2100
+Connection ~ 2850 2100
+Wire Wire Line
+	2750 2100 2850 2100
+Wire Wire Line
+	2550 2100 2750 2100
+Connection ~ 2750 2100
+$Comp
+L MCU_ST_STM32F1:STM32F103C8Tx U2
+U 1 1 5E490CEE
+P 2950 3600
+F 0 "U2" H 2900 2014 50  0000 C CNN
+F 1 "STM32F103C8Tx" H 2900 1923 50  0000 C CNN
+F 2 "Package_QFP:LQFP-48_7x7mm_P0.5mm" H 2350 2200 50  0001 R CNN
+F 3 "" H 2950 3600 50  0001 C CNN
+	1    2950 3600
+	1    0    0    -1
+$EndComp
+Wire Wire Line
+	2650 2450 2650 3500
+Wire Wire Line
+	2250 4300 3200 4300
+Wire Wire Line
+	3200 4300 3200 2800
+Wire Wire Line
+	3200 2800 3850 2800
+Wire Wire Line
+	4100 2800 4100 2700
+Wire Wire Line
+	4100 2700 3150 2700
+Wire Wire Line
+	3150 2700 3150 4200
+Wire Wire Line
+	3150 4200 2250 4200
+Wire Wire Line
+	4550 2800 4550 2650
+Wire Wire Line
+	4550 2650 3100 2650
+Wire Wire Line
+	3100 2650 3100 4100
+Wire Wire Line
+	3100 4100 2250 4100
+Wire Wire Line
+	2250 4000 3050 4000
+Wire Wire Line
+	3050 4000 3050 2600
+Wire Wire Line
+	3050 2600 4050 2600
+Wire Wire Line
+	4950 2600 4950 2800
+Connection ~ 4050 2600
+Wire Wire Line
+	4050 2600 4950 2600
+Wire Wire Line
+	5450 2450 5450 2800
+Wire Wire Line
+	2650 2450 5450 2450
+Wire Wire Line
+	5450 3200 4950 3200
 $EndSCHEMATC
